File: picstick_25k50_v1.brd (EAGLE design)
At the start: 50 x 20.4 mm, 16 parts, among them SW1 Reset, U1 PIC18F25K50-I/SP, X1 XTAL

Commit message: ...
Parts:
- JP1, JP2: value (none) -> CONN-14P; device LeoStick:FREETRONICS-JON_1X14 -> pinconn:CONN-14P
- moved JP1 16.5 mm to (31.8, 2.54)
- moved JP2 16.5 mm to (31.8, 20.3)
Connections:
- new net VSS: JP2.12
- net GND: no longer JP2.12
Changed lines of the file:
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@@
 <setting verticaltext="up"/>
 </settings>
-<grid distance="0.001" unitdist="inch" unit="inch" style="lines" multiple="1" display="no" altdistance="0.025" altunitdist="inch" altunit="inch"/>
+<grid distance="0.05" unitdist="inch" unit="inch" style="lines" multiple="2" display="yes" altdistance="0.005" altunitdist="inch" altunit="inch"/>
 <layers>
 <layer number="1" name="Top" color="4" fill="1" visible="yes" active="yes"/>
+<layer number="2" name="Route2" color="1" fill="3" visible="no" active="yes"/>
+<layer number="3" name="Route3" color="4" fill="3" visible="no" active="yes"/>
+<layer number="4" name="Route4" color="1" fill="4" visible="no" active="yes"/>
+<layer number="5" name="Route5" color="4" fill="4" visible="no" active="yes"/>
+<layer number="6" name="Route6" color="1" fill="8" visible="no" active="yes"/>
+<layer number="7" name="Route7" color="4" fill="8" visible="no" active="yes"/>
+<layer number="8" name="Route8" color="1" fill="2" visible="no" active="yes"/>
+<layer number="9" name="Route9" color="4" fill="2" visible="no" active="yes"/>
+<layer number="10" name="Route10" color="1" fill="7" visible="no" active="yes"/>
+<layer number="11" name="Route11" color="4" fill="7" visible="no" active="yes"/>
+<layer number="12" name="Route12" color="1" fill="5" visible="no" active="yes"/>
+<layer number="13" name="Route13" color="4" fill="5" visible="no" active="yes"/>
+<layer number="14" name="Route14" color="1" fill="6" visible="no" active="yes"/>
+<layer number="15" name="Route15" color="4" fill="6" visible="no" active="yes"/>
 <layer number="16" name="Bottom" color="1" fill="1" visible="yes" active="yes"/>
 <layer number="17" name="Pads" color="2" fill="1" visible="yes" active="yes"/>
 <layer number="18" name="Vias" color="2" fill="1" visible="yes" active="yes"/>
 <layer number="19" name="Unrouted" color="6" fill="1" visible="yes" active="yes"/>
-<layer number="20" name="Dimension" color="15" fill="1" visible="yes" active="yes"/>
-<layer number="21" name="tPlace" color="7" fill="1" visible="yes" active="yes"/>
-<layer number="22" name="bPlace" color="7" fill="1" visible="yes" active="yes"/>
+<layer number="20" name="Dimension" color="24" fill="1" visible="yes" active="yes"/>
+<layer number="21" name="tPlace" color="16" fill="1" visible="yes" active="yes"/>
+<layer number="22" name="bPlace" color="14" fill="1" visible="yes" active="yes"/>
 <layer number="23" name="tOrigins" color="15" fill="1" visible="yes" active="yes"/>
 <layer number="24" name="bOrigins" color="15" fill="1" visible="yes" active="yes"/>
 <layer number="25" name="tNames" color="7" fill="1" visible="yes" active="yes"/>
 <layer number="26" name="bNames" color="7" fill="1" visible="yes" active="yes"/>
-<layer number="27" name="tValues" color="7" fill="1" visible="no" active="yes"/>
-<layer number="28" name="bValues" color="7" fill="1" visible="no" active="yes"/>
+<layer number="27" name="tValues" color="7" fill="1" visible="yes" active="yes"/>
+<layer number="28" name="bValues" color="7" fill="1" visible="yes" active="yes"/>
 <layer number="29" name="tStop" color="7" fill="3" visible="no" active="yes"/>
 <layer number="30" name="bStop" color="7" fill="6" visible="no" active="yes"/>
@@
 <layer number="39" name="tKeepout" color="4" fill="11" visible="no" active="yes"/>
 <layer number="40" name="bKeepout" color="1" fill="11" visible="no" active="yes"/>
-<layer number="41" name="tRestrict" color="4" fill="10" visible="yes" active="yes"/>
-<layer number="42" name="bRestrict" color="1" fill="10" visible="yes" active="yes"/>
+<layer number="41" name="tRestrict" color="4" fill="10" visible="no" active="yes"/>
+<layer number="42" name="bRestrict" color="1" fill="10" visible="no" active="yes"/>
 <layer number="43" name="vRestrict" color="2" fill="10" visible="no" active="yes"/>
 <layer number="44" name="Drills" color="7" fill="1" visible="no" active="yes"/>
-<layer number="45" name="Holes" color="7" fill="1" visible="no" active="yes"/>
-<layer number="46" name="Milling" color="3" fill="1" visible="no" active="yes"/>
-<layer number="47" name="Measures" color="7" fill="1" visible="no" active="yes"/>
-<layer number="48" name="Document" color="7" fill="1" visible="no" active="yes"/>
-<layer number="49" name="Reference" color="7" fill="1" visible="no" active="yes"/>
+<layer number="45" name="Holes" color="7" fill="1" visible="yes" active="yes"/>
+<layer number="46" name="Milling" color="3" fill="1" visible="yes" active="yes"/>
+<layer number="47" name="Measures" color="7" fill="1" visible="yes" active="yes"/>
+<layer number="48" name="Document" color="7" fill="1" visible="yes" active="yes"/>
+<layer number="49" name="Reference" color="7" fill="1" visible="yes" active="yes"/>
 <layer number="50" name="dxf" color="7" fill="1" visible="no" active="yes"/>
-<layer number="51" name="tDocu" color="7" fill="1" visible="no" active="yes"/>
+<layer number="51" name="tDocu" color="6" fill="1" visible="yes" active="yes"/>
 <layer number="52" name="bDocu" color="7" fill="1" visible="no" active="yes"/>
 <layer number="91" name="Nets" color="2" fill="1" visible="no" active="no"/>
@@
 <param name="RoutingGrid" value="6.25mil"/>
 <param name="AutoGrid" value="1"/>
-<param name="Efforts" value="2"/>
+<param name="Efforts" value="0"/>
 <param name="TopRouterVariant" value="1"/>
 <param name="tpViaShape" value="round"/>
-<param name="PrefDir.1" value="a"/>
+<param name="PrefDir.1" value="|"/>
 <param name="PrefDir.2" value="0"/>
 <param name="PrefDir.3" value="0"/>
@@
 <param name="PrefDir.14" value="0"/>
 <param name="PrefDir.15" value="0"/>
-<param name="PrefDir.16" value="a"/>
+<param name="PrefDir.16" value="-"/>
 <param name="cfVia" value="8"/>
 <param name="cfNonPref" value="5"/>
@@
 <attribute name="VALUE" x="4.298" y="6.3508" size="0.4064" layer="27"/>
 </element>
-<element name="JP1" library="LeoStick" package="FREETRONICS-JON_1X14" value="" x="48.26" y="2.54" smashed="yes" rot="R180">
-<attribute name="NAME" x="49.53" y="3.5052" size="0.8128" layer="25" ratio="10" rot="R270"/>
-<attribute name="VALUE" x="42.672" y="4.699" size="1.27" layer="27" rot="R180"/>
-</element>
-<element name="JP2" library="LeoStick" package="FREETRONICS-JON_1X14" value="" x="48.26" y="20.32" smashed="yes" rot="R180">
-<attribute name="NAME" x="49.53" y="21.2344" size="0.8128" layer="25" ratio="10" rot="R270"/>
-<attribute name="VALUE" x="41.656" y="19.685" size="1.27" layer="27" rot="R180"/>
-</element>
+<element name="JP1" library="pinconn" package="CONN-14P" value="CONN-14P" x="31.75" y="2.54" rot="R180"/>
+<element name="JP2" library="pinconn" package="CONN-14P" value="CONN-14P" x="31.75" y="20.32" rot="R180"/>
 <element name="R4" library="rcl" package="0204/7" value="470R" x="35.8648" y="17.8308" smashed="yes" rot="R180">
 <attribute name="NAME" x="35.3568" y="18.3134" size="0.9906" layer="25" ratio="10" rot="R180"/>
@@
 <attribute name="OC_FARNELL" value="2305832" x="32.2072" y="11.43" size="1.778" layer="28" rot="MR90" display="off"/>
 <attribute name="NAME" x="48.9966" y="13.1064" size="0.8128" layer="26" ratio="10" rot="SMR90"/>
-<attribute name="VALUE" x="11.6586" y="6.2992" size="2.0828" layer="28" ratio="10" rot="SMR90"/>
 </element>
 <element name="R1" library="rcl" package="0204/7" value="470R" x="18.2626" y="17.8308" smashed="yes" rot="R180">
@@
 <contactref element="C3" pad="2"/>
 <contactref element="C4" pad="2"/>
-<contactref element="JP2" pad="12"/>
 <contactref element="SW1" pad="1"/>
 <contactref element="D2" pad="K"/>
@@
 <wire x1="23.7336" y1="17.8002" x2="21.2454" y2="20.2884" width="0.1778" layer="16"/>
 <wire x1="24.4992" y1="17.8002" x2="23.7336" y2="17.8002" width="0.1778" layer="16"/>
-<wire x1="20.4798" y1="20.2884" x2="20.32" y2="20.32" width="0.1778" layer="16"/>
 <wire x1="24.4992" y1="17.8002" x2="24.5872" y2="17.7546" width="0.1778" layer="16"/>
 <wire x1="30.8154" y1="8.8044" x2="30.8154" y2="7.656" width="0.1778" layer="16"/>
@@
 <wire x1="17.226" y1="18.9486" x2="13.398" y2="15.1206" width="0.1778" layer="1"/>
 <wire x1="18.9486" y1="18.9486" x2="17.226" y2="18.9486" width="0.1778" layer="1"/>
-<wire x1="20.32" y1="20.32" x2="18.9486" y2="18.9486" width="0.1778" layer="16"/>
 <wire x1="5.5506" y1="15.1206" x2="5.368" y2="14.9308" width="0.1778" layer="1"/>
 <wire x1="38.28" y1="11.2926" x2="39.237" y2="11.2926" width="0.1778" layer="1"/>
@@
 <vertex x="9.398" y="5.588"/>
 </polygon>
+<wire x1="20.4798" y1="20.2884" x2="20.2884" y2="20.2884" width="0.254" layer="16"/>
+<wire x1="20.2884" y1="20.2884" x2="18.9486" y2="18.9486" width="0.1778" layer="16"/>
 </signal>
 <signal name="RESET_SW">
@@
 <wire x1="16.269" y1="11.484" x2="16.1544" y2="11.4554" width="0.1778" layer="1"/>
 </signal>
+<signal name="VSS">
+<contactref element="JP2" pad="12"/>
+</signal>
 </signals>
