File: picstick_25k50_v1.sch (EAGLE design)
At the start: 16 parts, among them SW1 Reset, U1 PIC18F25K50-I/SP, X1 XTAL

Commit message: ...
Parts:
- JP1, JP2: value FREETRONICS-JON_M14 -> CONN-14P; device LeoStick:FREETRONICS-JON_M14 -> pinconn:CONN-14P
Connections:
- new net VSS: JP2.12
- net GND: no longer JP2.12
Other:
- note added: "ICSP"
- note added: "PGC / ICSPCLK"
- note added: "PGD / ICSPDAT"
- note added: "VPP"
- note removed: "ICSP Programming"
- moved on the sheet: C1, C2, C3, C4, D1, D2, R1, R2, R3, R4, SW1, U1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
